Commit message: update to traj

File: FetchArenaProject/Assets/URDF/ur10_with_gripper/ur10_with_gripper.urdf (robot description, URDF)
Before this commit: robot ur10_with_gripper, 22 links, 21 joints
Joints:
- joint shoulder_lift_joint: origin xyz=0.0 0.220941 0.0 rpy=0.0 1.5707963267948966 0.0 -> xyz=0.0 0.220941 0.0 rpy=0.0 0.0 0.0
- joint world_joint: origin xyz=1.653626 -0.0002509931 0.6694607 rpy=0.0 0.0 3.141592653589793 -> xyz=1.653626 0.0002509931 0.6694607 rpy=0.0 0.0 3.141592653589793
